Commit message: xacro fixes

File: urdf/jetank_arm.xacro (robot description, xacro)
@@ -1,4 +1,5 @@
 <?xml version="1.0"?>
 <robot xmlns:xacro="http://www.ros.org/wiki/xacro">
+<!--TODO FIX ROTATION PLACE-->
 <!-- Links -->
   <!-- Bearing -->
@@ -26,4 +27,5 @@
         <box size="${arm_camera_length} ${arm_camera_width} ${arm_camera_heigth}"/>
       </geometry>
+      <origin xyz="${arm_camera_length/2} 0 0" rpy="0 0 0"/>
     </visual>
   </link>
@@ -34,4 +36,5 @@
         <box size="${arm_long_length} ${arm_long_width} ${arm_long_heigth}"/>
       </geometry>
+      <origin xyz="${arm_long_length/2} 0 0" rpy="0 0 0"/>
     </visual>
   </link>
@@ -42,21 +45,22 @@
         <box size="${arm_short_length} ${arm_short_width} ${arm_short_heigth}"/>
       </geometry>
+      <origin xyz="${arm_long_length/2} 0 0" rpy="0 0 0"/>
     </visual>
   </link>
 <!-- Joints -->
   <!-- Arm bearing to chassis -->
-  <joint name="chassis_to_arm_bearing_joint" type="continuous">
+  <joint name="chassis_to_arm_bearing_joint" type="revolute">
     <parent link="chassis"/>
     <child link="arm_bearing_link"/>
     <origin xyz="${(chassis_length/2)-0.055} 0 ${(chassis_height/2)+(arm_bearing_height/2)}" rpy="0 0 0"/>
     <axis xyz="0 0 1"/>
+    <limit effort="10.0" lower="-1.0" upper="1.0" velocity="1.0"/>
   </joint>
   <!-- Arm base to arm bearing -->
-  <joint name="arm_base_to_arm_bearing_joint" type="revolute">
+  <joint name="arm_base_to_arm_bearing_joint" type="continuous">
     <parent link="arm_bearing_link"/>
     <child link="arm_base_link"/>
     <origin xyz="${((arm_base_length/2)-arm_bearing_radius)} 0 ${(arm_bearing_height/2)+(arm_base_heigth/2)}" rpy="0 0 0"/>
     <axis xyz="0 0 1"/>
-    <limit effort="10.0" lower="-1.0" upper="1.0" velocity="1.0"/>
   </joint>
   <!-- Camera to arm base joint -->
@@ -64,5 +68,5 @@
     <parent link="arm_base_link"/>
     <child link="arm_camera_link"/>
-    <origin xyz="${(arm_base_length/2)-0.01+(arm_camera_length/2)} 0 ${-(arm_base_heigth/2)+0.01}" rpy="0 0 0"/>
+    <origin xyz="${(arm_base_length/2)-0.01} 0 ${-(arm_base_heigth/2)+0.01}" rpy="0 0 0"/>
     <axis xyz="0 1 0"/>
     <limit effort="10.0" lower="-1.0" upper="1.0" velocity="1.0"/>
@@ -72,13 +76,13 @@
     <parent link="arm_base_link"/>
     <child link="arm_long_link"/>
-    <origin xyz="${(-arm_base_length/2)+0.03+(arm_long_length/2)} 0 ${arm_base_heigth/2-0.01}" rpy="0 0 0"/>
+    <origin xyz="${(-arm_base_length/2)+0.03} 0 ${arm_base_heigth/2-0.01}" rpy="0 0 0"/>
     <axis xyz="0 1 0"/>
     <limit effort="10.0" lower="-1.0" upper="1.0" velocity="1.0"/>
   </joint>
   <!-- Short link to long link joint -->
-  <joint name="arm_base_to_short_joint" type="revolute">
+  <joint name="arm_long_to_short_joint" type="revolute">
     <parent link="arm_long_link"/>
     <child link="arm_short_link"/>
-    <origin xyz="${(arm_long_length/2)-0.01+(arm_short_length/2)} 0 0" rpy="0 0 0"/>
+    <origin xyz="${(arm_long_length)-0.01} 0 0" rpy="0 0 0"/>
     <axis xyz="0 1 0"/>
     <limit effort="10.0" lower="-1.0" upper="1.0" velocity="1.0"/>

File: urdf/jetank_wheel.xacro (robot description, xacro)
@@ -23,5 +23,5 @@
       <child link="${prefix}_wheel"/>
       <origin xyz="${x} ${y} ${z}" rpy="0 0 0"/>
-      <axis xyz="0 0 1"/>
+      <axis xyz="0 1 0"/>
     </joint>
   </xacro:macro>

Commit message: gripper xacro

File: urdf/jetank_arm.xacro (robot description, xacro)
@@ -1,10 +1,8 @@
 <?xml version="1.0"?>
 <robot xmlns:xacro="http://www.ros.org/wiki/xacro">
-<!--TODO FIX ROTATION PLACE-->
 <!-- Links -->
   <!-- Bearing -->
   <link name="arm_bearing_link">
     <visual>
-      <!-- <origin xyz="${(chassis_length/2)-(arm_base_length/2)} 0 ${(chassis_height/2)+arm_base_heigth+arm_bearing_height}" rpy="0 0 0"/> -->
       <geometry>
         <cylinder length="${arm_bearing_height}" radius="${arm_bearing_radius}"/>
@@ -15,5 +13,4 @@
   <link name="arm_base_link">
     <visual>
-      <!-- <origin xyz="${(chassis_length/2)-(arm_base_length/2)} 0 ${(chassis_height/2)+arm_base_heigth+arm_bearing_height}" rpy="0 0 0"/> -->
       <geometry>
         <box size="${arm_base_length} ${arm_base_width} ${arm_base_heigth}"/>

File: urdf/properties.xacro (robot description, xacro)
@@ -20,6 +20,14 @@
   <xacro:property name="arm_long_width" value="0.055"/>
   <xacro:property name="arm_long_heigth" value="0.025"/>
-  <xacro:property name="arm_short_length" value="0.115"/>
+  <xacro:property name="arm_short_length" value="0.09"/>
   <xacro:property name="arm_short_width" value="0.045"/>
   <xacro:property name="arm_short_heigth" value="0.02"/>
+  <!-- Gripper parameters -->
+  <xacro:property name="gripper_base_length" value="0.04"/>
+  <xacro:property name="gripper_base_width" value="0.08"/>
+  <xacro:property name="gripper_base_heigth" value="0.06"/>
+  <xacro:property name="gripper_finger_length" value="0.06"/>
+  <xacro:property name="gripper_finger_width" value="0.03"/>
+  <xacro:property name="gripper_finger_heigth" value="0.025"/>
+  <xacro:property name="gripper_finger_range" value="0.02"/>
 </robot>

Commit message: Fix urdf to pase positions

File: urdf/jetank_arm.xacro (robot description, xacro)
@@ -73,5 +73,5 @@
     <parent link="arm_base_link"/>
     <child link="arm_long_link"/>
-    <origin xyz="${(-arm_base_length/2)+0.03} 0 ${arm_base_heigth/2-0.01}" rpy="0 0 0"/>
+    <origin xyz="${(-arm_base_length/2)+0.03} 0 ${arm_base_heigth/2-0.01}" rpy="0 -1.57079632679 0"/>
     <axis xyz="0 1 0"/>
     <limit effort="10.0" lower="-1.0" upper="1.0" velocity="1.0"/>
@@ -81,5 +81,5 @@
     <parent link="arm_long_link"/>
     <child link="arm_short_link"/>
-    <origin xyz="${(arm_long_length)-0.01} 0 0" rpy="0 0 0"/>
+    <origin xyz="${(arm_long_length)-0.01} 0 0" rpy="0 1.57079632679 0"/>
     <axis xyz="0 1 0"/>
     <limit effort="10.0" lower="-1.0" upper="1.0" velocity="1.0"/>

File: urdf/jetank_gripper.xacro (robot description, xacro)
@@ -45,5 +45,5 @@
     <limit lower="0" upper="${gripper_finger_range}" effort="10.0" velocity="1.0"/>
     <axis xyz="0 1 0"/>
-    <mimic joint="left_finger_joint" multiplier="-1.0" offset="0.0"/>
+    <mimic joint="left_finger_joint" multiplier="1.0" offset="0.0"/>
   </joint>
 </robot>

Commit message: wip camera calib

File: urdf/jetank_arm.xacro (robot description, xacro)
@@ -19,5 +19,5 @@
   </link>
   <!-- Camera Link -->
-  <link name="arm_camera_link">
+  <link name="camera_link">
     <visual>
       <geometry>
@@ -64,5 +64,5 @@
   <joint name="arm_base_to_camera_joint" type="revolute">
     <parent link="arm_base_link"/>
-    <child link="arm_camera_link"/>
+    <child link="camera_link"/>
     <origin xyz="${(arm_base_length/2)-0.01} 0 ${-(arm_base_heigth/2)+0.01}" rpy="0 0 0"/>
     <axis xyz="0 1 0"/>
