Commit message: wip urdf

File: urdf/jetank.xacro (robot description, xacro)
@@ -1,4 +1,7 @@
 <?xml version="1.0"?>
 <robot name="jetank" xmlns:xacro="http://www.ros.org/wiki/xacro">
+  <xacro:include filename="$(find robot_main)/urdf/properties.xacro"/>
+  <xacro:include filename="$(find robot_main)/urdf/jetank_wheel.xacro"/>
+  <xacro:include filename="$(find robot_main)/urdf/jetank_arm.xacro"/>
   <!-- Base link -->
   <link name="base_link" />
@@ -22,3 +25,10 @@
     <child link="chassis"/>
   </joint>
+      <!-- Instantiate wheels -->
+  <xacro:wheel prefix="left_front" x="${((chassis_length/2)-(0.02+wheel_radius))}" y="${-((chassis_width / 2)+(wheel_length/2))}" z="${wheel_radius}"/>
+  <xacro:wheel prefix="right_front" x="${((chassis_length/2)-(0.02+wheel_radius))}" y="${((chassis_width / 2)+(wheel_length/2))}" z="${wheel_radius}"/>
+  <xacro:wheel prefix="left_middle" x="0" y="${-((chassis_width / 2)+(wheel_length/2))}" z="${wheel_radius}"/>
+  <xacro:wheel prefix="right_middle" x="0" y="${((chassis_width / 2)+(wheel_length/2))}" z="${wheel_radius}"/>
+  <xacro:wheel prefix="left_back" x="${-((chassis_length/2)-(0.02+wheel_radius))}" y="${-((chassis_width / 2)+(wheel_length/2))}" z="${wheel_radius}"/>
+  <xacro:wheel prefix="right_back" x="${-((chassis_length/2)-(0.02+wheel_radius))}" y="${((chassis_width / 2)+(wheel_length/2))}" z="${wheel_radius}"/>
 </robot>

File: urdf/jetank_wheel.xacro (robot description, xacro)
@@ -26,10 +26,3 @@
     </joint>
   </xacro:macro>
-    <!-- Instantiate wheels -->
-  <xacro:wheel prefix="left_front" x="${((chassis_length/2)-(0.02+wheel_radius))}" y="${-((chassis_width / 2)+(wheel_length/2))}" z="${wheel_radius}"/>
-  <xacro:wheel prefix="right_front" x="${((chassis_length/2)-(0.02+wheel_radius))}" y="${((chassis_width / 2)+(wheel_length/2))}" z="${wheel_radius}"/>
-  <xacro:wheel prefix="left_middle" x="0" y="${-((chassis_width / 2)+(wheel_length/2))}" z="${wheel_radius}"/>
-  <xacro:wheel prefix="right_middle" x="0" y="${((chassis_width / 2)+(wheel_length/2))}" z="${wheel_radius}"/>
-  <xacro:wheel prefix="left_back" x="${-((chassis_length/2)-(0.02+wheel_radius))}" y="${-((chassis_width / 2)+(wheel_length/2))}" z="${wheel_radius}"/>
-  <xacro:wheel prefix="right_back" x="${-((chassis_length/2)-(0.02+wheel_radius))}" y="${((chassis_width / 2)+(wheel_length/2))}" z="${wheel_radius}"/>
 </robot>

File: urdf/properties.xacro (robot description, xacro)
@@ -1,5 +1,5 @@
 <?xml version="1.0" ?>
 <robot xmlns:xacro="http://www.ros.org/wiki/xacro">
-  <!-- Basic parameters -->
+  <!-- Chassis parameters -->
   <xacro:property name="chassis_length" value="0.2"/>
   <xacro:property name="chassis_width" value="0.1"/>
@@ -8,3 +8,16 @@
   <xacro:property name="wheel_length" value="0.05"/>
   <xacro:property name="ground_clearance" value="0.01"/>
+  <!-- Arm parameters -->
+  <xacro:property name="arm_base_length" value="0.070"/>
+  <xacro:property name="arm_base_width" value="0.045"/>
+  <xacro:property name="arm_base_heigth" value="0.075"/>
+  <xacro:property name="arm_camera_length" value="0.045"/>
+  <xacro:property name="arm_camera_width" value="0.055"/>
+  <xacro:property name="arm_camera_heigth" value="0.025"/>
+  <xacro:property name="arm_long_length" value="0.12"/>
+  <xacro:property name="arm_long_width" value="0.055"/>
+  <xacro:property name="arm_long_heigth" value="0.025"/>
+  <xacro:property name="arm_short_length" value="0.115"/>
+  <xacro:property name="arm_short_width" value="0.045"/>
+  <xacro:property name="arm_short_heigth" value="0.02`"/>
 </robot>

Commit message: added arm xacro, still without gripper though

File: urdf/jetank.xacro (robot description, xacro)
@@ -9,5 +9,5 @@
   <link name="chassis">
     <visual>
-      <origin xyz="0 0 ${ground_clearance+(chassis_height/2)}" />
+      <!-- <origin xyz="0 0 ${ground_clearance+(chassis_height/2)}" /> -->
       <geometry>
         <box size="${chassis_length} ${chassis_width} ${chassis_height}"/>
@@ -15,5 +15,5 @@
     </visual>
     <collision>
-      <origin xyz="0.0 0.0 ${(ground_clearance+(chassis_height/2))}"/>
+      <!-- <origin xyz="0.0 0.0 ${(ground_clearance+(chassis_height/2))}"/> -->
       <geometry>
         <box size="${chassis_length} ${chassis_width} ${chassis_height}"/>
@@ -24,11 +24,12 @@
     <parent link="base_link"/>
     <child link="chassis"/>
+    <origin xyz="0.0 0.0 ${(ground_clearance+(chassis_height/2))}"/>
   </joint>
       <!-- Instantiate wheels -->
-  <xacro:wheel prefix="left_front" x="${((chassis_length/2)-(0.02+wheel_radius))}" y="${-((chassis_width / 2)+(wheel_length/2))}" z="${wheel_radius}"/>
-  <xacro:wheel prefix="right_front" x="${((chassis_length/2)-(0.02+wheel_radius))}" y="${((chassis_width / 2)+(wheel_length/2))}" z="${wheel_radius}"/>
-  <xacro:wheel prefix="left_middle" x="0" y="${-((chassis_width / 2)+(wheel_length/2))}" z="${wheel_radius}"/>
-  <xacro:wheel prefix="right_middle" x="0" y="${((chassis_width / 2)+(wheel_length/2))}" z="${wheel_radius}"/>
-  <xacro:wheel prefix="left_back" x="${-((chassis_length/2)-(0.02+wheel_radius))}" y="${-((chassis_width / 2)+(wheel_length/2))}" z="${wheel_radius}"/>
-  <xacro:wheel prefix="right_back" x="${-((chassis_length/2)-(0.02+wheel_radius))}" y="${((chassis_width / 2)+(wheel_length/2))}" z="${wheel_radius}"/>
+  <xacro:wheel prefix="left_front" x="${((chassis_length/2)-(0.02+wheel_radius))}" y="${-((chassis_width / 2)+(wheel_length/2))}" z="${-wheel_radius}"/>
+  <xacro:wheel prefix="right_front" x="${((chassis_length/2)-(0.02+wheel_radius))}" y="${((chassis_width / 2)+(wheel_length/2))}" z="${-wheel_radius}"/>
+  <xacro:wheel prefix="left_middle" x="0" y="${-((chassis_width / 2)+(wheel_length/2))}" z="${-wheel_radius}"/>
+  <xacro:wheel prefix="right_middle" x="0" y="${((chassis_width / 2)+(wheel_length/2))}" z="${-wheel_radius}"/>
+  <xacro:wheel prefix="left_back" x="${-((chassis_length/2)-(0.02+wheel_radius))}" y="${-((chassis_width / 2)+(wheel_length/2))}" z="${-wheel_radius}"/>
+  <xacro:wheel prefix="right_back" x="${-((chassis_length/2)-(0.02+wheel_radius))}" y="${((chassis_width / 2)+(wheel_length/2))}" z="${-wheel_radius}"/>
 </robot>

File: urdf/jetank_arm.xacro (robot description, xacro)
@@ -2,7 +2,17 @@
 <robot xmlns:xacro="http://www.ros.org/wiki/xacro">
 <!-- Links -->
+  <!-- Bearing -->
+  <link name="arm_bearing_link">
+    <visual>
+      <!-- <origin xyz="${(chassis_length/2)-(arm_base_length/2)} 0 ${(chassis_height/2)+arm_base_heigth+arm_bearing_height}" rpy="0 0 0"/> -->
+      <geometry>
+        <cylinder length="${arm_bearing_height}" radius="${arm_bearing_radius}"/>
+      </geometry>
+    </visual>
+  </link>
   <!-- Base Link -->
   <link name="arm_base_link">
     <visual>
+      <!-- <origin xyz="${(chassis_length/2)-(arm_base_length/2)} 0 ${(chassis_height/2)+arm_base_heigth+arm_bearing_height}" rpy="0 0 0"/> -->
       <geometry>
         <box size="${arm_base_length} ${arm_base_width} ${arm_base_heigth}"/>
@@ -35,9 +45,16 @@
   </link>
 <!-- Joints -->
-  <!-- Arm base to chassis joint -->
-  <joint name="chassis_to_arm_base_joint" type="revolute">
+  <!-- Arm bearing to chassis -->
+  <joint name="chassis_to_arm_bearing_joint" type="continuous">
     <parent link="chassis"/>
+    <child link="arm_bearing_link"/>
+    <origin xyz="${(chassis_length/2)-0.055} 0 ${(chassis_height/2)+(arm_bearing_height/2)}" rpy="0 0 0"/>
+    <axis xyz="0 0 1"/>
+  </joint>
+  <!-- Arm base to arm bearing -->
+  <joint name="arm_base_to_arm_bearing_joint" type="revolute">
+    <parent link="arm_bearing_link"/>
     <child link="arm_base_link"/>
-    <origin xyz="${(chassis_length/2)-0.055} 0 ${chassis_height/2}" rpy="0 0 0"/>
+    <origin xyz="${((arm_base_length/2)-arm_bearing_radius)} 0 ${(arm_bearing_height/2)+(arm_base_heigth/2)}" rpy="0 0 0"/>
     <axis xyz="0 0 1"/>
     <limit effort="10.0" lower="-1.0" upper="1.0" velocity="1.0"/>
@@ -47,5 +64,5 @@
     <parent link="arm_base_link"/>
     <child link="arm_camera_link"/>
-    <origin xyz="${(arm_base_length/2)-0.01} 0 ${-arm_base_heigth/2+0.1}" rpy="0 0 0"/>
+    <origin xyz="${(arm_base_length/2)-0.01+(arm_camera_length/2)} 0 ${-(arm_base_heigth/2)+0.01}" rpy="0 0 0"/>
     <axis xyz="0 1 0"/>
     <limit effort="10.0" lower="-1.0" upper="1.0" velocity="1.0"/>
@@ -55,5 +72,5 @@
     <parent link="arm_base_link"/>
     <child link="arm_long_link"/>
-    <origin xyz="${(arm_base_length/2)-0.01} 0 ${-arm_base_heigth/2+0.1}" rpy="0 0 0"/>
+    <origin xyz="${(-arm_base_length/2)+0.03+(arm_long_length/2)} 0 ${arm_base_heigth/2-0.01}" rpy="0 0 0"/>
     <axis xyz="0 1 0"/>
     <limit effort="10.0" lower="-1.0" upper="1.0" velocity="1.0"/>
@@ -63,5 +80,5 @@
     <parent link="arm_long_link"/>
     <child link="arm_short_link"/>
-    <origin xyz="${(arm_base_length/2)-0.01} 0 ${-arm_base_heigth/2+0.1}" rpy="0 0 0"/>
+    <origin xyz="${(arm_long_length/2)-0.01+(arm_short_length/2)} 0 0" rpy="0 0 0"/>
     <axis xyz="0 1 0"/>
     <limit effort="10.0" lower="-1.0" upper="1.0" velocity="1.0"/>

File: urdf/jetank_test.urdf (robot description, URDF)
Before this commit: robot jetank, 12 links, 11 joints
Links:
- link arm_short_link: geometry visual box size=0.115 0.045 0.02
Joints:
- joint arm_base_to_long_joint: origin xyz=0.025 0 0.0625 rpy=0 0 0 -> xyz=-0.005 0 -0.0625 rpy=0 0 0
- joint arm_base_to_short_joint: origin xyz=0.025 0 0.0625 rpy=0 0 0 -> xyz=0.05 0 0 rpy=0 0 0

File: urdf/properties.xacro (robot description, xacro)
@@ -9,4 +9,6 @@
   <xacro:property name="ground_clearance" value="0.01"/>
   <!-- Arm parameters -->
+  <xacro:property name="arm_bearing_radius" value="0.02"/>
+  <xacro:property name="arm_bearing_height" value="0.01"/>
   <xacro:property name="arm_base_length" value="0.070"/>
   <xacro:property name="arm_base_width" value="0.045"/>
@@ -20,4 +22,4 @@
   <xacro:property name="arm_short_length" value="0.115"/>
   <xacro:property name="arm_short_width" value="0.045"/>
-  <xacro:property name="arm_short_heigth" value="0.02`"/>
+  <xacro:property name="arm_short_heigth" value="0.02"/>
 </robot>

Commit message: Finalizer urdf

File: urdf/jetank.xacro (robot description, xacro)
@@ -4,4 +4,5 @@
   <xacro:include filename="$(find robot_main)/urdf/jetank_wheel.xacro"/>
   <xacro:include filename="$(find robot_main)/urdf/jetank_arm.xacro"/>
+  <xacro:include filename="$(find robot_main)/urdf/jetank_gripper.xacro"/>
   <!-- Base link -->
   <link name="base_link" />

File: urdf/jetank_gripper.xacro (robot description, xacro)
@@ -13,9 +13,8 @@
 <!-- Joints -->
   <!-- Gripper base to arm -->
-  <joint name="arm_base_to_arm_bearing_joint" type="fixed">
+  <joint name="gripper_base_to_arm_joint" type="fixed">
     <parent link="arm_short_link"/>
     <child link="gripper_base_link"/>
     <origin xyz="${arm_short_length+(gripper_base_length/2)} ${0.01} ${(gripper_base_heigth/2)}" rpy="0 0 0"/>
-    <!-- <axis xyz="0 0 1"/> -->
   </joint>
   <xacro:macro name="finger" params="prefix x y z direction">
@@ -27,5 +26,5 @@
       </visual>
     </link>
-    <joint name="${prefix}_wheel_joint" type="prismatic">
+    <joint name="${prefix}_finger_joint" type="prismatic">
       <parent link="gripper_base_link"/>
       <child link="${prefix}_finger_link"/>
@@ -35,5 +34,5 @@
     </joint>
   </xacro:macro>
-  <xacro:finger prefix="left" x="${}" y="${}" z="${}" direction="-1"/>
-  <xacro:finger prefix="right" x="${}" y="${}" z="${}" direction="1"/>
+  <xacro:finger prefix="left" x="${gripper_finger_length/2}" y="${(gripper_finger_range+(gripper_finger_width/2))-0.01}" z="0" direction="-1"/>
+  <xacro:finger prefix="right" x="${gripper_finger_length/2}" y="${-(gripper_finger_range+(gripper_finger_width/2))-0.01}" z="0" direction="1"/>
 </robot>

File: urdf/properties.xacro (robot description, xacro)
@@ -29,5 +29,5 @@
   <xacro:property name="gripper_finger_length" value="0.06"/>
   <xacro:property name="gripper_finger_width" value="0.03"/>
-  <xacro:property name="gripper_finger_heigth" value="0.025"/>
+  <xacro:property name="gripper_finger_heigth" value="0.02"/>
   <xacro:property name="gripper_finger_range" value="0.02"/>
 </robot>

Commit message: Update URDF for stereo camera

File: urdf/jetank.xacro (robot description, xacro)
@@ -5,4 +5,5 @@
   <xacro:include filename="$(find robot_main)/urdf/jetank_arm.xacro"/>
   <xacro:include filename="$(find robot_main)/urdf/jetank_gripper.xacro"/>
+  <xacro:include filename="$(find robot_main)/urdf/jetank_camera.xacro"/>
   <!-- Base link -->
   <link name="base_link" />

File: urdf/jetank_arm.xacro (robot description, xacro)
@@ -19,5 +19,5 @@
   </link>
   <!-- Camera Link -->
-  <link name="camera_link">
+  <link name="camera_base_link">
     <visual>
       <geometry>
@@ -64,5 +64,5 @@
   <joint name="arm_base_to_camera_joint" type="revolute">
     <parent link="arm_base_link"/>
-    <child link="camera_link"/>
+    <child link="camera_base_link"/>
     <origin xyz="${(arm_base_length/2)-0.01} 0 ${-(arm_base_heigth/2)+0.01}" rpy="0 0 0"/>
     <axis xyz="0 1 0"/>

File: urdf/jetank_gripper.xacro (robot description, xacro)
@@ -16,5 +16,5 @@
     <parent link="arm_short_link"/>
     <child link="gripper_base_link"/>
-    <origin xyz="${arm_short_length+(gripper_base_length/2)} ${0.01} ${(gripper_base_heigth/2)}" rpy="0 0 0"/>
+    <origin xyz="${arm_short_length+(gripper_base_length/2)} ${0.01} ${(gripper_base_heigth/2)-(arm_short_heigth/2)}" rpy="0 0 0"/>
   </joint>
   <link name="left_finger_link">
@@ -28,5 +28,5 @@
     <parent link="gripper_base_link"/>
     <child link="left_finger_link"/>
-    <origin xyz="${gripper_finger_length/2} ${(gripper_finger_range+(gripper_finger_width/2))-0.01} 0" rpy="0 0 0"/>
+    <origin xyz="${gripper_finger_length/2} ${(gripper_finger_range+(gripper_finger_width/2))-0.01} ${-gripper_finger_heigth}" rpy="0 0 0"/>
     <limit lower="0" upper="${gripper_finger_range}" effort="10.0" velocity="1.0"/>
     <axis xyz="0 -1 0"/>
@@ -42,5 +42,5 @@
     <parent link="gripper_base_link"/>
     <child link="right_finger_link"/>
-    <origin xyz="${gripper_finger_length/2} ${-(gripper_finger_range+(gripper_finger_width/2))-0.01} 0" rpy="0 0 0"/>
+    <origin xyz="${gripper_finger_length/2} ${-(gripper_finger_range+(gripper_finger_width/2))-0.01} ${-gripper_finger_heigth}" rpy="0 0 0"/>
     <limit lower="0" upper="${gripper_finger_range}" effort="10.0" velocity="1.0"/>
     <axis xyz="0 1 0"/>

File: urdf/properties.xacro (robot description, xacro)
@@ -11,5 +11,5 @@
   <xacro:property name="arm_bearing_radius" value="0.02"/>
   <xacro:property name="arm_bearing_height" value="0.01"/>
-  <xacro:property name="arm_base_length" value="0.070"/>
+  <xacro:property name="arm_base_length" value="0.045"/>
   <xacro:property name="arm_base_width" value="0.045"/>
   <xacro:property name="arm_base_heigth" value="0.075"/>
@@ -31,3 +31,10 @@
   <xacro:property name="gripper_finger_heigth" value="0.02"/>
   <xacro:property name="gripper_finger_range" value="0.02"/>
+  <!-- Camera parameters -->
+  <xacro:property name="camera_base_length" value="0.0016"/>
+  <xacro:property name="camera_base_width" value="0.085"/>
+  <xacro:property name="camera_base_heigth" value="0.025"/>
+  <xacro:property name="camera_radius" value="0.008"/>
+  <xacro:property name="camera_heigth" value="0.022"/>
+  <xacro:property name="camera_dist" value="0.03"/>
 </robot>
