Commit message: clearing local changes for change to ros2

File: urdf/jetank_camera.xacro (robot description, xacro)
@@ -37,5 +37,5 @@
     <parent link="camera_base_plate_link"/>
     <child link="camera_left_link"/>
-    <origin xyz="${camera_heigth/2} ${camera_dist} ${0.0}" rpy="0 -1.57079632679 0"/>
+    <origin xyz="${camera_heigth/2} ${camera_dist} ${0.0}" rpy="0 1.57079632679 0"/>
   </joint>
   <!-- Camera right to base -->
@@ -43,5 +43,5 @@
     <parent link="camera_base_plate_link"/>
     <child link="camera_right_link"/>
-    <origin xyz="${camera_heigth/2} ${-camera_dist} ${0.0}" rpy="0 -1.57079632679 0"/>
+    <origin xyz="${camera_heigth/2} ${-camera_dist} ${0.0}" rpy="0 1.57079632679 0"/>
   </joint>
 </robot>
